File: hardware/dc.kicad_pcb (KiCad board)
At the start: 4 copper layers, 80 x 80 mm, 89 parts, among them P1 CON-SENSOR2, P2 DEBUG, P3 BOOT, P4 OUT, P5 GPIO, P6 IN, Q1 CSD19533Q5A, Q2 CSD19533Q5A, Q3 CSD19533Q5A, Q4 CSD19533Q5A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

Commit message: new hardware version
Other:
- board text added: "DC 2.1"
- board text removed: "DC 2.0"
Changed lines of the file:
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@@
-(kicad_pcb (version 20171130) (host pcbnew 5.1.6-c6e7f7d~86~ubuntu20.04.1)
+(kicad_pcb (version 20171130) (host pcbnew 5.1.6-c6e7f7d~87~ubuntu20.04.1)
   (general
     (thickness 1.6)
@@
     (effects (font (size 0.8 0.8) (thickness 0.15)))
   )
-  (gr_text "DC\n2.0" (at 136.7 140.5 90) (layer F.SilkS)
+  (gr_text "DC\n2.1" (at 136.7 140.5 90) (layer F.SilkS)
     (effects (font (size 1.5 1.5) (thickness 0.25)))
   )
@@
   (via (at 139 171.2) (size 0.5) (drill 0.2) (layers F.Cu B.Cu) (net 2))
   (via (at 138.2 171.2) (size 0.5) (drill 0.2) (layers F.Cu B.Cu) (net 2))
-  (via (at 138.3 159.7) (size 0.5) (drill 0.2) (layers F.Cu B.Cu) (net 8))
-  (via (at 137.7 159.7) (size 0.5) (drill 0.2) (layers F.Cu B.Cu) (net 8))
-  (via (at 137.1 159.7) (size 0.5) (drill 0.2) (layers F.Cu B.Cu) (net 8))
-  (via (at 136.5 159.7) (size 0.5) (drill 0.2) (layers F.Cu B.Cu) (net 8))
-  (via (at 139 164.3) (size 0.5) (drill 0.2) (layers F.Cu B.Cu) (net 8))
+  (via (at 137.4 171.2) (size 0.5) (drill 0.2) (layers F.Cu B.Cu) (net 2))
+  (via (at 137.4 170.5) (size 0.5) (drill 0.2) (layers F.Cu B.Cu) (net 2))
+  (via (at 137.4 169.8) (size 0.5) (drill 0.2) (layers F.Cu B.Cu) (net 2))
+  (via (at 137.4 169.1) (size 0.5) (drill 0.2) (layers F.Cu B.Cu) (net 2))
+  (via (at 137.4 168.4) (size 0.5) (drill 0.2) (layers F.Cu B.Cu) (net 2))
+  (via (at 137.4 167.7) (size 0.5) (drill 0.2) (layers F.Cu B.Cu) (net 2))
+  (via (at 137.4 167) (size 0.5) (drill 0.2) (layers F.Cu B.Cu) (net 2))
+  (via (at 137.4 166.2) (size 0.5) (drill 0.2) (layers F.Cu B.Cu) (net 2))
+  (via (at 138.2 165.7) (size 0.5) (drill 0.2) (layers F.Cu B.Cu) (net 2))
   (segment (start 98.25 107.6) (end 98.35 107.7) (width 0.7) (layer F.Cu) (net 3))
   (segment (start 98.25 105.4) (end 98.25 107.6) (width 0.7) (layer F.Cu) (net 3))
@@
   (segment (start 110.95 107.35) (end 108.5 104.9) (width 0.2) (layer F.Cu) (net 7))
   (segment (start 117.9 107.35) (end 110.95 107.35) (width 0.2) (layer F.Cu) (net 7))
+  (via (at 138.3 159.7) (size 0.5) (drill 0.2) (layers F.Cu B.Cu) (net 8))
+  (via (at 137.7 159.7) (size 0.5) (drill 0.2) (layers F.Cu B.Cu) (net 8))
+  (via (at 137.1 159.7) (size 0.5) (drill 0.2) (layers F.Cu B.Cu) (net 8))
+  (via (at 136.5 159.7) (size 0.5) (drill 0.2) (layers F.Cu B.Cu) (net 8))
+  (via (at 139 164.3) (size 0.5) (drill 0.2) (layers F.Cu B.Cu) (net 8))
   (via (at 84.1 167.3) (size 0.8) (drill 0.5) (layers F.Cu B.Cu) (net 8))
   (segment (start 81.4 167.3) (end 83.534315 167.3) (width 0.9) (layer In2.Cu) (net 8))
@@
   (via (at 137.1 164.9) (size 0.5) (drill 0.2) (layers F.Cu B.Cu) (net 8))
   (via (at 136.5 164.9) (size 0.5) (drill 0.2) (layers F.Cu B.Cu) (net 8))
+  (segment (start 92.8 160.925) (end 93.9525 159.7725) (width 0.25) (layer F.Cu) (net 8))
+  (segment (start 92.8 162.3) (end 92.8 160.925) (width 0.25) (layer F.Cu) (net 8))
+  (segment (start 92.8 163.675) (end 93.9525 164.8275) (width 0.25) (layer F.Cu) (net 8))
+  (segment (start 92.8 162.3) (end 92.8 163.675) (width 0.25) (layer F.Cu) (net 8))
   (segment (start 100.4507 107.1507) (end 100.4507 107.925) (width 0.2) (layer F.Cu) (net 10))
   (segment (start 99.5 105.4) (end 99.5 106.2) (width 0.2) (layer F.Cu) (net 10))
@@
   (segment (start 119.65 121.45) (end 119.65 120.9) (width 0.25) (layer F.Cu) (net 43))
   (segment (start 117.275 121.95) (end 117.525 121.7) (width 0.25) (layer F.Cu) (net 43))
-  (via (at 137.4 171.2) (size 0.5) (drill 0.2) (layers F.Cu B.Cu) (net 2))
-  (via (at 137.4 170.5) (size 0.5) (drill 0.2) (layers F.Cu B.Cu) (net 2))
-  (via (at 137.4 169.8) (size 0.5) (drill 0.2) (layers F.Cu B.Cu) (net 2))
-  (via (at 137.4 169.1) (size 0.5) (drill 0.2) (layers F.Cu B.Cu) (net 2))
-  (via (at 137.4 168.4) (size 0.5) (drill 0.2) (layers F.Cu B.Cu) (net 2))
-  (via (at 137.4 167.7) (size 0.5) (drill 0.2) (layers F.Cu B.Cu) (net 2))
-  (via (at 137.4 167) (size 0.5) (drill 0.2) (layers F.Cu B.Cu) (net 2))
-  (via (at 137.4 166.2) (size 0.5) (drill 0.2) (layers F.Cu B.Cu) (net 2))
-  (via (at 138.2 165.7) (size 0.5) (drill 0.2) (layers F.Cu B.Cu) (net 2))
-  (segment (start 92.8 160.925) (end 93.9525 159.7725) (width 0.25) (layer F.Cu) (net 8))
-  (segment (start 92.8 162.3) (end 92.8 160.925) (width 0.25) (layer F.Cu) (net 8))
-  (segment (start 92.8 163.675) (end 93.9525 164.8275) (width 0.25) (layer F.Cu) (net 8))
-  (segment (start 92.8 162.3) (end 92.8 163.675) (width 0.25) (layer F.Cu) (net 8))
   (segment (start 124.35 149.9) (end 124.3 149.85) (width 0.25) (layer F.Cu) (net 44))
   (via (at 125.799998 149.3) (size 0.5) (drill 0.2) (layers F.Cu B.Cu) (net 44))
