File: hardware/dc.kicad_pcb (KiCad board)
At the start: 4 copper layers, 80 x 80 mm, 89 parts, among them P1 CON-SENSOR2, P2 DEBUG, P3 BOOT, P4 OUT, P5 GPIO, P6 IN, Q1 CSD19533Q5A, Q2 CSD19533Q5A, Q3 CSD19533Q5A, Q4 CSD19533Q5A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

Commit message: added logos to back silkscreen
Parts:
- added G***: LOGO, kicad-libraries:Logo_CoMCU, B.Cu at (99.5, 143.6)
- added VAL: WEEE_7mm, kicad-libraries:WEEE_7mm, B.Cu at (92.2, 144.0)
- added VAL: CE_5mm, kicad-libraries:CE_5mm, B.Cu at (107.5, 143.5)

Commit message: changed input voltage silkscreen
Other:
- board text added: "Input 6-36V"
Changed lines of the file:
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@@
-(kicad_pcb (version 20171130) (host pcbnew 5.1.6-c6e7f7d~87~ubuntu20.04.1)
+(kicad_pcb (version 20171130) (host pcbnew "(5.1.4)-1")
   (general
     (thickness 1.6)
@@
     (effects (font (size 2 2) (thickness 0.25)))
   )
-  (gr_text "Input\n6-45V" (at 65.05 172.3) (layer F.SilkS)
+  (gr_text "Input\n6-36V" (at 65.05 172.3) (layer F.SilkS)
     (effects (font (size 1 1) (thickness 0.15)))
   )
