File: hardware/performance-dc.kicad_pcb (KiCad board)
At the start: 4 copper layers, 80 x 80 mm, 91 parts, among them P1 CON-SENSOR2, P2 DEBUG, P3 BOOT, P4 OUT, P5 GPIO, P6 IN, Q1 CSD19533Q5A, Q2 CSD19533Q5A, Q3 CSD19533Q5A, Q4 CSD19533Q5A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

Commit message: specify processor
Parts:
- U1: value XMC1??? -> XMC1302

Commit message: specify drv8701p
Parts:
- U6: value DRV8701 -> DRV8701P
